Commit message: Adapt robot arm package to ROS 2 Jazzy

File: urdf/right arm Walter.urdf (robot description, URDF)
Before this commit: robot right arm Walter, 4 links, 3 joints
Links:
- added link world
- link base_link: geometry collision mesh filename=package://right_arm_walter/meshes/base_link.STL; visual mesh filename=package://right_arm_walter/meshes/base_link.STL
- link elbow_Link: geometry collision mesh filename=package://right_arm_walter/meshes/elbow_Link.STL; visual mesh filename=package://right_arm_walter/meshes/elbow_Link.STL
- link pitch_Link: geometry collision mesh filename=package://right_arm_walter/meshes/pitch_Link.STL; visual mesh filename=package://right_arm_walter/meshes/pitch_Link.STL
- link roll_Link: geometry collision mesh filename=package://right_arm_walter/meshes/roll_Link.STL; visual mesh filename=package://right_arm_walter/meshes/roll_Link.STL
Joints:
- added joint world_to_base: type fixed, parent world, child base_link, origin xyz=0 0 0.5 rpy=0 -1.5708 0
- joint elbow_joint: limit lower=0 upper=0 effort=0 velocity=0 -> lower=-1.5708 upper=0 effort=5 velocity=1.0
- joint pitch_joint: limit lower=0 upper=0 effort=0 velocity=0 -> lower=-1.5708 upper=1.5708 effort=5 velocity=1.0
- joint roll_joint: limit lower=0 upper=0 effort=0 velocity=0 -> lower=-1.5708 upper=0 effort=5 velocity=1.0

Commit message: Update robot arm package for ROS 2 Jazzy

File: urdf/right arm Walter.urdf (robot description, URDF)
Before this commit: robot right arm Walter, 5 links, 4 joints
Joints:
- joint elbow_joint: axis 0 0 -1 -> 0 0 1; limit lower=-1.5708 upper=0 effort=5 velocity=1.0 -> lower=0 upper=1.5708 effort=5 velocity=1.0
- joint pitch_joint: axis 0 0 -1 -> 0 0 1
- joint roll_joint: axis 0 0 -1 -> 0 0 1; limit lower=-1.5708 upper=0 effort=5 velocity=1.0 -> lower=0 upper=1.5708 effort=5 velocity=1.0
